Commit message: override srdf after move_group include
and update the SRDF-config

File: prbt_default_application/config/prbt.srdf.xacro (robot description, xacro)
@@ -1,17 +1,13 @@
 <?xml version="1.0" ?>
 <robot name="prbt" xmlns:xacro="http://www.ros.org/wiki/xacro">
-  <!-- parameter -->
-  <xacro:arg name="gripper" default=""/>
-  <xacro:property name="gripper" value="$(arg gripper)"/>
-  <xacro:arg name="prefix" default="prbt_"/>
   <!--VIRTUAL JOINT: Purpose: this element defines a virtual joint between a robot link and an
                      external frame of reference (considered fixed with respect to the robot)-->
-  <virtual_joint name="FixedBase" type="fixed" parent_frame="world" child_link="$(arg prefix)base_link" />
+  <virtual_joint name="FixedBase" type="fixed" parent_frame="world" child_link="table" />
   <!-- robot manipulator -->
   <xacro:include filename="$(find prbt_moveit_config)/config/prbt_manipulator.srdf.xacro" />
-  <xacro:prbt_manipulator prefix="$(arg prefix)"/>
-  <!-- has gripper -->
-  <xacro:unless value="${not gripper}">
-    <xacro:include filename="$(find prbt_${gripper}_support)/config/${gripper}.srdf.xacro" />
-  </xacro:unless>
+  <xacro:prbt_manipulator prefix="prbt_"/>
+  <!-- add gripper -->
+  <!-- <xacro:include filename="$(find prbt_pg70_support)/config/pg70.srdf.xacro" /> -->
+  <!-- you can add disabled collisions here -->
+  <!-- <disable_collisions link1="prbt_flange" link2="my_custom_gripper" reason="Adjacent" /> -->
 </robot>

File: prbt_default_application/urdf/my_first_application.xacro (robot description, xacro)
@@ -41,5 +41,5 @@
     <child link="pnoz"/>
   </joint>
-  <!-- connect the added tcp and the flange with a joint (tutorial 2)-->
+  <!-- connect the added tcp and the flange with a joint -->
   <joint name="prbt_fixed_joint_tcp" type="fixed">
     <origin rpy="0 0 0" xyz="0 0 0.05"/>
